File: hardware/main-board/nes-cpu.sch (KiCad schematic (older format))
At the start: 37 parts, among them SW1 NES Reset, U10 74HCT00, U11 PCA9564, U3 74LVC1404, U4 RP2A03, U5 74HCT138, U6 LM4889, U7 AS6C6264, U8 MCP40D17, U9 AT28C64B, Y1 21.5 MHz

Commit message: Update hardware project to support KiCad v5
This change does all the necessary symbol remapping and file re-saving
so that KiCad v5 is now cleanly supported going forward. Hopefully there
are no actual changes of consequence introduced by this diff.
Parts:
- C10, C11, C13, C15, C16, C17, C18, C19, C5, C7, C8, C9: symbol C -> Device:C
- C12, C14, C6: symbol CP -> Device:CP
- R10, R11, R12, R13, R14, R17, R5, R6, R7, R8, R9: symbol R -> Device:R
- SW1: symbol SW_Push -> Switch:SW_Push
- U10: symbol 74HCT00 -> 74xx:74HCT00
- U11: symbol PCA9564 -> nes:PCA9564
- U3: symbol SN74LVC1404 -> nes:SN74LVC1404
- U4: symbol RP2A03 -> nes:RP2A03
- U5: symbol 74HCT138 -> nes:74HCT138
- U6: symbol LM4889 -> nes:LM4889
- U7: symbol AS6C6264 -> nes:AS6C6264
- U8: symbol MCP40D17 -> nes:MCP40D17
- U9: symbol AT28C64B -> nes:AT28C64B
- Y1: symbol Crystal -> Device:Crystal
