File: hardware/main-board/nes.sch (KiCad schematic (older format))
At the start: 14 parts, among them J1 Power Jack, J2 Input Board, J3 Speaker, U1 R-78E5.0-0.5, U2 R-78E3.3-0.5

Commit message: Update hardware project to support KiCad v5
This change does all the necessary symbol remapping and file re-saving
so that KiCad v5 is now cleanly supported going forward. Hopefully there
are no actual changes of consequence introduced by this diff.
Parts:
- C1, C2, C3, C4: symbol C -> Device:C
- D1: symbol D -> Device:D
- J1: symbol Barrel_Jack -> Connector:Barrel_Jack_Switch
- J2: symbol Conn_01x06 -> Connector_Generic:Conn_01x06
- J3: symbol Conn_01x02 -> Connector_Generic:Conn_01x02
- R1, R2, R3, R4: symbol R -> Device:R
- U1: symbol R-78E5.0-0.5 -> Regulator_Switching:R-78E5.0-0.5
- U2: symbol R-78E3.3-0.5 -> Regulator_Switching:R-78E3.3-0.5
